File: kicad-project/atmega2560.kicad_sch (KiCad schematic)
At the start: 1 part

Commit message: hw: update
Parts:
- added C?: (no value), Capacitor_SMD:C_0805_2012Metric, symbol Device:C
- added C?: 1u, Capacitor_SMD:C_0805_2012Metric, symbol Device:C
- added C? (x2): 18p, Capacitor_SMD:C_0603_1608Metric, symbol Device:C
- added C? (x2): 100n, Capacitor_SMD:C_0603_1608Metric, symbol Device:C
- added J?: Conn_02x08_Counter_Clockwise, Connector_PinHeader_2.54mm:PinHeader_2x05_P2.54mm_Vertical, symbol Connector_Generic:Conn_02x05_Counter_Clockwise
- added J?: Conn_02x03_Counter_Clockwise, Connector_PinHeader_2.54mm:PinHeader_2x03_P2.54mm_Vertical, symbol Connector_Generic:Conn_02x03_Counter_Clockwise
- added R? (x3): 10k, Resistor_SMD:R_0603_1608Metric, symbol Device:R
- added R?: (no value), Resistor_SMD:R_0603_1608Metric, symbol Device:R
- added SW?: HOME_SW, Button_Switch_THT:SW_PUSH_6mm, symbol Switch:SW_Push
- added SW?: EN_SW, Button_Switch_THT:SW_PUSH_6mm, symbol Switch:SW_Push
- added SW?: RST_SW, Button_Switch_THT:SW_PUSH_6mm, symbol Switch:SW_Push
- added Y?: 12MHz, Crystal:Crystal_SMD_3225-4Pin_3.2x2.5mm, symbol Device:Crystal_GND24
Connections:
- net +5V: now also C?.1, J?.1 (Pin_1), J?.1 (Pin_1), R?.1, R?.1, R?.1
- net GND: now also C?.2, C?.2, C?.2, C?.2, C?.2, C?.2, J?.2 (Pin_2), J?.2 (Pin_2), SW?.2, SW?.2, SW?.2, Y?.2, Y?.4
- net ~{RESET}: now reaches U?.30 (~{RESET})
- net ~{RESET}: now also R?.2, SW?.1
- new net AREF: C?.1
- new net EXT_ADC0: J?.4 (Pin_4)
- new net EXT_ADC1: J?.6 (Pin_6)
- new net GPIO1: J?.9 (Pin_9)
- new net GPIO2: J?.7 (Pin_7)
- new net GPIO3: J?.10 (Pin_10)
- new net GPIO4: J?.8 (Pin_8)
- new net I2C1_SCL: J?.3 (Pin_3), J?.5 (Pin_5)
- new net I2C1_SDA: J?.3 (Pin_3), J?.5 (Pin_5)
- new net SWCLK: J?.6 (Pin_6)
- new net SWDIO: J?.4 (Pin_4)
- new net XIN: C?.1, Y?.1
- new net XOUT: R?.2
- new net iXOUT: C?.1, R?.1, Y?.3
- new net ~{EN_SW}: C?.1, R?.2, SW?.1
- new net ~{HOME_SW}: C?.1, R?.2, SW?.1
Other:
- note added: "Crystal"
- note added: "Debug"
- note added: "Expansion"
- note added: "Home Switch"
- note added: "Motor Enable Switch"
- note added: "Reset Switch"
- note added: "https://docs.arduino.cc/static/de2dcffb754755b0fb1ede880bd153ba/schematics.pdf"
- note added: "ma il quarzo ha un'orientazione?"

Commit message: hw: add esp8266
Parts:
- added C? (x2): 100n, Capacitor_SMD:C_0603_1608Metric, symbol Device:C
- C?: value (none) -> 100n
- C? (x2): value 18p -> (none)
- R?: value (none) -> 1M
- Y?: value 12MHz -> (none)
Connections:
- net +5V: now also U?.100 (AVCC), C?.1, C?.1
- net GND: now also C?.2, C?.2
- net XIN renamed XTAL1
- net XOUT renamed XTAL2
- net iXOUT renamed iXTAL2
Other:
- note added: "pin a vcc 10 31 61 80"

Commit message: hw: change to rp2040
Parts:
- removed U?: ATmega2560-16A, Package_QFP:TQFP-100_14x14mm_P0.5mm, symbol MCU_Microchip_ATmega:ATmega2560-16A
- added C? (x10): 100n, Capacitor_SMD:C_0603_1608Metric, symbol Device:C
- added C? (x2): 1u, Capacitor_SMD:C_0805_2012Metric, symbol Device:C
- added C?: DNP 100n, Capacitor_SMD:C_0603_1608Metric, symbol Device:C
- added R? (x2): 27R, Resistor_SMD:R_0603_1608Metric, symbol Device:R
- added R?: DNP 10k, Resistor_SMD:R_0603_1608Metric, symbol Device:R
- added R?: 1k, Resistor_SMD:R_0603_1608Metric, symbol Device:R
- added SW?: PRG_SW, Button_Switch_THT:SW_PUSH_6mm, symbol Switch:SW_Push
- added U?: W25Q16JVSS, Package_SO:SOIC-8_5.23x5.23mm_P1.27mm, symbol Memory_Flash:W25Q32JVSS
- added U?: RP2040, ppse_2021:RP2040-Hand-Solder, symbol AA_PPSE_2021:RP2040
- C? (x2): value (none) -> 22p
- Y?: value (none) -> 16MHz; footprint Crystal:Crystal_SMD_3225-4Pin_3.2x2.5mm -> Crystal:Crystal_SMD_HC49-SD; symbol Device:Crystal_GND24 -> Device:Crystal
Connections:
- net EXT_ADC0: now also U?.40 (GPIO28/ADC2)
- net EXT_ADC1: now also U?.41 (GPIO29/ADC3)
- net GND: now also C?.2, C?.2, C?.2, C?.2, C?.2, C?.2, C?.2, C?.2, C?.2, C?.2, C?.2, C?.2, C?.2, SW?.2, U?.19 (TESTEN), U?.4 (GND), U?.57 (GND); no longer Y?.2, Y?.4
- net GPIO1: now also U?.3 (GPIO1)
- net GPIO2: now also U?.4 (GPIO2)
- net GPIO3: now also U?.5 (GPIO3)
- net GPIO4: now also U?.6 (GPIO4)
- net I2C1_SCL: now also U?.30 (GPIO19)
- net I2C1_SDA: now also U?.29 (GPIO18)
- net SWCLK: now also U?.24 (SWCLK)
- net SWDIO: now also U?.25 (SWDIO)
- net iXTAL2: now also Y?.2; no longer Y?.3
- net ~{EN_SW}: now also U?.7 (GPIO5)
- net ~{HOME_SW}: now also U?.8 (GPIO6)
- net ~{RESET}: now also U?.26 (RUN)
- net +5V renamed +3V3
- net +3V3: now also C?.1, C?.1, C?.1, C?.1, C?.1, C?.1, C?.1, C?.1, C?.1, C?.1, R?.1, U?.1 (IOVDD), U?.10 (IOVDD), U?.22 (IOVDD), U?.33 (IOVDD), U?.42 (IOVDD), U?.43 (ADC_AVDD), U?.44 (VREG_VIN), U?.48 (USB_VDD), U?.49 (IOVDD), U?.8 (VCC)
- new net +1V1: C?.1, C?.1, C?.1, U?.23 (DVDD), U?.45 (VREG_VOUT), U?.50 (DVDD)
- new net ACC_INT: U?.32 (GPIO21)
- new net Buzzer: U?.2 (GPIO0)
- new net CMP_DRDY: U?.31 (GPIO20)
- new net FLASH_CLK: U?.52 (QSPI_SCLK), U?.6 (CLK)
- new net FLASH_D0: U?.5 (DI(IO0)), U?.53 (QSPI_SD0)
- new net FLASH_D1: U?.2 (DO(IO1)), U?.55 (QSPI_SD1)
- new net FLASH_D2: U?.3 (IO2), U?.54 (QSPI_SD2)
- new net FLASH_D3: U?.51 (QSPI_SD3), U?.7 (IO3)
- new net GPS_EN: U?.34 (GPIO22)
- new net GPS_TIMEPULSE: U?.35 (GPIO23)
- new net I_{PANEL}: U?.39 (GPIO27/ADC1)
- new net LED_B: U?.12 (GPIO9)
- new net LED_G: U?.9 (GPIO7)
- new net LED_R: U?.11 (GPIO8)
- new net M1_W11: U?.17 (GPIO14)
- new net M1_W12: U?.18 (GPIO15)
- new net M1_W21: U?.27 (GPIO16)
- new net M1_W22: U?.28 (GPIO17)
- new net M2_W11: U?.13 (GPIO10)
- new net M2_W12: U?.14 (GPIO11)
- new net M2_W21: U?.15 (GPIO12)
- new net M2_W22: U?.16 (GPIO13)
- new net UART1_RX: U?.37 (GPIO25)
- new net UART1_TX: U?.36 (GPIO24)
- new net USB_D+: R?.2
- new net USB_D-: R?.2
- new net V_{PANEL}: U?.38 (GPIO26/ADC0)
- new net XIN: U?.20 (XIN)
- new net XOUT: U?.21 (XOUT)
- new net iUSB_D+: R?.1, U?.47 (USB_DP)
- new net iUSB_D-: R?.1, U?.46 (USB_DM)
- new net ~{FLASH_CS}: R?.2, R?.2, U?.1 (~{CS}), U?.56 (QSPI_SS_N)
- new net ~{USB_BOOT}: R?.1, SW?.1
Other:
- note added: "Flash"
- note added: "If CS=0 => Mass storage (Program) If CS=1 => Read content (Run)"
- note added: "MCU Filters"
- note added: "Make sure to place all capacitors close to their respective pins"
- note added: "Place resistors close to pin"
- note added: "pin a vcc 31 61 80"
- note removed: "pin a vcc 10 31 61 80"
- moved on the sheet: C?, J?, R?, SW?

Commit message: hw: change power management and drivers
Parts:
- removed C?: 100n, Capacitor_SMD:C_0805_2012Metric, symbol Device:C
- removed C?: 1u, Capacitor_SMD:C_0805_2012Metric, symbol Device:C
- removed C? (x3): 100n, Capacitor_SMD:C_0603_1608Metric, symbol Device:C
- removed R?: 10k, Resistor_SMD:R_0603_1608Metric, symbol Device:R
- removed SW?: HOME_SW, Button_Switch_THT:SW_PUSH_6mm, symbol Switch:SW_Push
- removed U?: RP2040, ppse_2021:RP2040-Hand-Solder, symbol AA_PPSE_2021:RP2040
- added U?: (no value), symbol HSD:RP2040
Connections:
- net XTAL1 is gone; now on net XIN: C?.1, Y?.1
- net XTAL2 is gone; now on net XOUT: R?.2
- net +1V1: now also U?.23 (DVDD), U?.45 (VREG_VOUT), U?.50 (DVDD)
- net +3V3: now also U?.1 (IOVDD), U?.10 (IOVDD), U?.22 (IOVDD), U?.33 (IOVDD), U?.42 (IOVDD), U?.43 (ADC_AVDD), U?.44 (VREG_VIN), U?.48 (USB_VDD), U?.49 (IOVDD); no longer J?.1 (Pin_1), J?.1 (Pin_1), R?.1, R?.1
- net ACC_INT: now also U?.32 (GPIO21)
- net Buzzer: now also U?.2 (GPIO0)
- net CMP_DRDY: now also U?.31 (GPIO20)
- net FLASH_CLK: now also U?.52 (QSPI_SCLK)
- net FLASH_D0: now also U?.53 (QSPI_SD0)
- net FLASH_D1: now also U?.55 (QSPI_SD1)
- net FLASH_D2: now also U?.54 (QSPI_SD2)
- net FLASH_D3: now also U?.51 (QSPI_SD3)
- net GND: now also U?.19 (TESTEN), U?.57 (GND)
- net GPIO1: now also U?.3 (GPIO1)
- net GPIO2: now also U?.4 (GPIO2)
- net GPIO3: now also U?.5 (GPIO3)
- net GPIO4: now also U?.6 (GPIO4)
- net GPS_EN: now also U?.34 (GPIO22)
- net GPS_TIMEPULSE: now also U?.35 (GPIO23)
- net I2C1_SCL: now also U?.30 (GPIO19)
- net I2C1_SDA: now also U?.29 (GPIO18)
- net LED_B: now also U?.12 (GPIO9)
- net LED_G: now also U?.9 (GPIO7)
- net LED_R: now also U?.11 (GPIO8)
- net M1_W11: now also U?.17 (GPIO14)
- net M1_W12: now also U?.18 (GPIO15)
- net M1_W21: now also U?.27 (GPIO16)
- net M1_W22: now also U?.28 (GPIO17)
- net M2_W11: now also U?.13 (GPIO10)
- net M2_W12: now also U?.14 (GPIO11)
- net M2_W21: now also U?.15 (GPIO12)
- net M2_W22: now also U?.16 (GPIO13)
- net UART1_RX: now also U?.37 (GPIO25)
- net UART1_TX: now also U?.36 (GPIO24)
- net XIN: now also U?.20 (XIN)
- net XOUT: now also U?.21 (XOUT)
- net iUSB_D+: now also U?.47 (USB_DP)
- net iUSB_D-: now also U?.46 (USB_DM)
- net ~{EN_SW}: now also U?.7 (GPIO5)
- net ~{FLASH_CS}: now also U?.56 (QSPI_SS_N)
- net ~{RESET}: now also U?.26 (RUN)
- net iXTAL2 renamed iXOUT
- new net +5V: J?.1 (Pin_1), J?.1 (Pin_1), R?.1, R?.1
- new net xxx: U?.8 (GPIO6)
- no-connect marks 0 -> 6
Other:
- note added: "Place R_{termination} close to rp2040 pins"
- note removed: "Home Switch"
- note removed: "Make sure to place all capacitors close to their respective pins"
- note removed: "https://docs.arduino.cc/static/de2dcffb754755b0fb1ede880bd153ba/schematics.pdf"
- note removed: "ma il quarzo ha un'orientazione?"
- note removed: "pin a vcc 31 61 80"
- moved on the sheet: C?, R?, SW?, U?, Y?

Commit message: Bipolar pins
Parts:
- U?: value (none) -> RP2040; footprint (none) -> HSD:RP2040-Hand-Solder
Changed lines of the file:
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@@
       (effects (font (size 1.27 1.27)) (justify left))
     )
-    (property "Value" "" (id 1) (at 54.61 36.83 0)
+    (property "Value" "RP2040" (id 1) (at 54.61 36.83 0)
       (effects (font (size 1.27 1.27)) (justify left))
     )
-    (property "Footprint" "" (id 2) (at 96.52 88.9 0)
+    (property "Footprint" "HSD:RP2040-Hand-Solder" (id 2) (at 96.52 88.9 0)
       (effects (font (size 1.27 1.27)) hide)
     )
