File: kicad-project/bipolars.kicad_sch (KiCad schematic)
At the start: 28 parts, among them J10 Conn_01x08_Female, J11 Conn_01x08_Female, J12 Conn_01x08_Female, J13 Conn_01x04_Male, J14 Conn_01x04_Male, J3 Conn_01x08_Female, J4 Conn_01x08_Female, J5 Conn_01x08_Female, J6 Conn_01x08_Female, J7 Conn_01x04_Male, J8 Conn_01x04_Male, J9 Conn_01x08_Female, U5 A4988SETTR-T

Commit message: hw: finish schematic, PS i2c R_pull-up wrong
Parts:
- removed C29, C31: 0.1u, symbol Device:C
- removed C30, C32: 0.22u, symbol Device:C
- removed C33: 100u, symbol Device:C_Polarized
- removed J10, J11, J12, J3, J4, J5, J6, J9: Conn_01x08_Female, symbol Connector:Conn_01x08_Female
- removed R15: 10k, symbol Device:R
- removed R16: R_Variable, symbol Device:R_Variable
- removed R17: 100K, symbol Device:R
- removed R18, R19: 0.1, symbol Device:R
- removed R20: R, symbol Device:R
- removed U5: A4988SETTR-T, QFN50P500X500X90-29N, symbol A4988:A4988SETTR-T
- added J4, J5, J6, J9: Conn_01x02_Female, Connector_PinHeader_2.54mm:PinHeader_1x02_P2.54mm_Vertical, symbol Connector:Conn_01x02_Female
- added U5, U6, U7, U8: A4988_Shield, HSD:A4988_Shield, symbol HSD:A4988_Shield
- C25, C26, C27, C28: footprint (none) -> Capacitor_SMD:CP_Elec_6.3x5.3
- J13, J14, J7, J8: footprint (none) -> Connector_PinHeader_2.54mm:PinHeader_1x04_P2.54mm_Vertical
Connections:
- net +12V: now also U5.16 (VMOT), U6.16 (VMOT), U7.16 (VMOT), U8.16 (VMOT)
- net +3V3: now also U5.10 (VDD), U5.2 (MS1), U5.3 (MS2), U5.4 (MS3), U6.10 (VDD), U6.2 (MS1), U6.3 (MS2), U6.4 (MS3), U7.10 (VDD), U7.2 (MS1), U7.3 (MS2), U7.4 (MS3), U8.10 (VDD), U8.2 (MS1), U8.3 (MS2), U8.4 (MS3)
- net DIR_A: now also U5.8 (DIR)
- net DIR_B: now also U7.8 (DIR)
- net DIR_C: now also U6.8 (DIR)
- net DIR_D: now also U8.8 (DIR)
- net EN_MOTORS: now also U5.1 (~{ENABLE}), U6.1 (~{ENABLE}), U7.1 (~{ENABLE}), U8.1 (~{ENABLE})
- net GND: now also J4.2 (Pin_2), J5.2 (Pin_2), J6.2 (Pin_2), J9.2 (Pin_2), U5.15 (GND), U5.9 (GND), U6.15 (GND), U6.9 (GND), U7.15 (GND), U7.9 (GND), U8.15 (GND), U8.9 (GND)
- net MA_1A: now also U5.12 (1A)
- net MA_1B: now also U5.11 (1B)
- net MA_2A: now also U5.13 (2A)
- net MA_2B: now also U5.14 (2B)
- net MB_1A: now also U7.12 (1A)
- net MB_1B: now also U7.11 (1B)
- net MB_2A: now also U7.13 (2A)
- net MB_2B: now also U7.14 (2B)
- net MC_1A: now also U6.12 (1A)
- net MC_1B: now also U6.11 (1B)
- net MC_2A: now also U6.13 (2A)
- net MC_2B: now also U6.14 (2B)
- net MD_1A: now also U8.12 (1A)
- net MD_1B: now also U8.11 (1B)
- net MD_2A: now also U8.13 (2A)
- net MD_2B: now also U8.14 (2B)
- net STEP_A: now also U5.7 (STEP)
- net STEP_B: now also U7.7 (STEP)
- net STEP_C: now also U6.7 (STEP)
- net STEP_D: now also U8.7 (STEP)
- new net: U5.5 (~{RST}), U5.6 (~{SLEEP})
- new net: U7.5 (~{RST}), U7.6 (~{SLEEP})
- new net: U6.5 (~{RST}), U6.6 (~{SLEEP})
- new net: U8.5 (~{RST}), U8.6 (~{SLEEP})
- new net LS1: J4.1 (Pin_1)
- new net LS2: J5.1 (Pin_1)
- new net LS3: J6.1 (Pin_1)
- new net LS4: J9.1 (Pin_1)
- no-connect marks 1 -> 0
Other:
- note added: "Limit switches"
- note removed: "1/16 step"
- note removed: "Vref=Imax*8*Rs con 1.3A -> 1V 90%*1.3=1.17A -> 0.935V"
- note removed: "capire che cosa fare con ROSC"
- moved on the sheet: C25, C26, C27, C28, J13, J14, J7, J8
