File: kicad-project/bipolars.kicad_sch (KiCad schematic)
At the start: 28 parts, among them J10 Conn_01x08_Female, J11 Conn_01x08_Female, J12 Conn_01x08_Female, J13 Conn_01x04_Male, J14 Conn_01x04_Male, J3 Conn_01x08_Female, J4 Conn_01x08_Female, J5 Conn_01x08_Female, J6 Conn_01x08_Female, J7 Conn_01x04_Male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

Commit message: hw: finish schematic
Parts:
- removed C29, C31: 0.1u, symbol Device:C
- removed C30, C32: 0.22u, symbol Device:C
- removed C33: 100u, symbol Device:C_Polarized
- removed R15: 10k, symbol Device:R
- removed R16: R_Variable, symbol Device:R_Variable
- removed R17: 100K, symbol Device:R
- removed R18, R19: 0.1, symbol Device:R
- removed R20: R, symbol Device:R
- removed U5: A4988SETTR-T, QFN50P500X500X90-29N, symbol A4988:A4988SETTR-T
- C25, C26, C27, C28: footprint (none) -> Capacitor_SMD:CP_Elec_6.3x5.3
- J13, J14, J7, J8: footprint (none) -> Connector_PinHeader_2.54mm:PinHeader_1x04_P2.54mm_Vertical
Connections:
- no-connect marks 1 -> 0
Other:
- note added: "TODO simbolo con footprint 6 pin di spazio da 2.54mm 12.7mm"
- note removed: "1/16 step"
- note removed: "Vref=Imax*8*Rs con 1.3A -> 1V 90%*1.3=1.17A -> 0.935V"
- note removed: "capire che cosa fare con ROSC"
