File: kicad-project/peripherals.kicad_sch (KiCad schematic)
At the start: 26 parts, among them J15 Conn_01x04, J16 Conn_01x02_Female, J17 Conn_01x02_Female, J18 Conn_02x04_Odd_Even, J19 Conn_01x02_Female, J20 Conn_01x02_Female, Q1 S8050, Q2 S8050, Q3 S8050, Q4 S8050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

Commit message: hw: finish schematic
Parts:
- added D11: 1N4148WS, Diode_SMD:D_SOD-323, symbol Device:D
- D6: footprint LED_SMD:LED_RGB_1210 -> LED_SMD:LED_RGB_5050-6
- J15: footprint Connector_PinHeader_2.54mm:PinHeader_1x04_P2.54mm_Vertical_SMD_Pin1Left -> Connector_PinHeader_2.54mm:PinHeader_1x04_P2.54mm_Vertical
- J16, J17, J19, J20: footprint (none) -> Connector_PinHeader_2.54mm:PinHeader_1x02_P2.54mm_Vertical
- J18: footprint (none) -> Connector_PinHeader_2.54mm:PinHeader_2x04_P2.54mm_Vertical
- Q1, Q2, Q3, Q4: value S8050 -> BC847B
- R27: value 10k -> 5k; footprint (none) -> Resistor_SMD:R_0603_1608Metric
- R28: value 47k -> DNP; footprint (none) -> Resistor_SMD:R_0603_1608Metric
- R30, R31, R32: footprint (none) -> Resistor_SMD:R_0603_1608Metric
- SW4: footprint Button_Switch_THT:SW_PUSH_6mm_H4.3mm -> Button_Switch_SMD:SW_Push_1P1T_NO_CK_KMR2
Connections:
- net +3V3: now also D11.1 (K)
- net iBuzzer: no longer names the net of BZ1.2 (+), Q4.3 (C), R29.2
- net iBuzzer: now also D11.2 (A)
- net ~{iLED_B}: no longer names the net of D6.3 (BK), R26.2
- net ~{iLED_G}: no longer names the net of D6.2 (GK), R24.2
- net ~{iLED_R}: no longer names the net of D6.1 (RK), R22.2
Other:
- moved on the sheet: R22, R24, R26, R27
