File: kicad-project/power.kicad_sch (KiCad schematic)
At the start: 32 parts, among them J1 Screw_Terminal_01x02, J2 USB_C_Receptacle_USB2.0, U1 TPS563201, U2 AMS1117-3.3

Commit message: hw: finish schematic
Parts:
- removed FB1: FerriteBead, Inductor_SMD:L_0603_1608Metric, symbol Device:FerriteBead
- C1, C2, C3, C7, C8: Voltage 16V -> (none)
- C4, C5, C6: Voltage 6V3 -> (none)
- D1: footprint (none) -> Diode_SMD:D_SOD-123
- D2: footprint Diode_SMD:D_SMA -> Diode_SMD:D_SOD-123
- D3: value SMA S1B -> GS1504FL; footprint Diode_SMD:D_SMA -> Diode_SMD:D_SOD-123F
- D4: footprint (none) -> Diode_SMD:D_SOD-323
- F1: value 2929L-LF075 -> 2920L075; footprint (none) -> Fuse:Fuse_2920_7451Metric
- F2: footprint (none) -> Fuse:Fuse_1206_3216Metric
- J1: footprint (none) -> TerminalBlock_RND:TerminalBlock_RND_205-00001_1x02_P5.00mm_Horizontal
- J2: footprint (none) -> HSD:USB-C-USB4105-GF-A-120
- L1: footprint ppse_2021:Inductor -> (none)
- R1, R2, R3: footprint (none) -> Resistor_SMD:R_0603_1608Metric
- R5: Tolerance 1% -> (none)
Connections:
- net VBUS_FILTERED is gone; now on net VBUS: D4.2 (A)
Other:
- note added: "0603 C fino a 100n 0805 C da 1u in sù"
- note removed: "TUTTI I FOORPRINT SONO DA VERIFICARE/AGGIUNGERE"
Changed lines of the file:
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@@
     (stroke (width 0) (type default) (color 0 0 0 0))
   )
-  (wire (pts (xy 45.085 105.41) (xy 53.34 105.41))
+  (wire (pts (xy 45.085 105.41) (xy 83.82 105.41))
     (stroke (width 0) (type default) (color 0 0 0 0))
   )
@@
   )
   (wire (pts (xy 245.11 44.45) (xy 248.92 44.45))
-    (stroke (width 0) (type default) (color 0 0 0 0))
-  )
-  (wire (pts (xy 60.96 105.41) (xy 83.82 105.41))
     (stroke (width 0) (type default) (color 0 0 0 0))
   )
@@
     (effects (font (size 2.5 2.5) (thickness 0.5994) bold) (justify right bottom))
   )
+  (text "0603 C fino a 100n\n0805 C da 1u in sù" (at 107.95 67.31 0)
+    (effects (font (size 1.27 1.27)) (justify left bottom))
+  )
   (text "6A\n" (at 43.18 68.58 0)
     (effects (font (size 1.27 1.27)) (justify left bottom))
@@
     (effects (font (size 2.5 2.5) (thickness 0.6) bold) (justify left bottom))
   )
-  (text "TUTTI I FOORPRINT SONO DA VERIFICARE/AGGIUNGERE\n\n" (at 134.62 119.38 0)
-    (effects (font (size 4 4) (thickness 0.8) bold) (justify left bottom))
-  )
   (label "SW_BST" (at 168.91 52.07 0)
     (effects (font (size 1.27 1.27)) (justify left bottom))
@@
   )
   (label "SW_VIN" (at 139.7 44.45 0)
-    (effects (font (size 1.27 1.27)) (justify left bottom))
-  )
-  (label "VBUS_FILTERED" (at 63.5 105.41 0)
     (effects (font (size 1.27 1.27)) (justify left bottom))
   )
@@
       (effects (font (size 1.27 1.27)) (justify left))
     )
-    (property "Footprint" "" (id 2) (at 52.07 48.26 0)
+    (property "Footprint" "Diode_SMD:D_SOD-123" (id 2) (at 52.07 48.26 0)
       (effects (font (size 1.27 1.27)) hide)
     )
@@
     (property "Reference" "J1" (id 0) (at 21.59 38.1 0))
     (property "Value" "Screw_Terminal_01x02" (id 1) (at 21.59 40.64 0))
-    (property "Footprint" "" (id 2) (at 21.59 46.99 0)
+    (property "Footprint" "TerminalBlock_RND:TerminalBlock_RND_205-00001_1x02_P5.00mm_Horizontal" (id 2) (at 21.59 46.99 0)
       (effects (font (size 1.27 1.27)) hide)
     )
@@
     (property "Reference" "J2" (id 0) (at 29.845 97.79 0))
     (property "Value" "USB_C_Receptacle_USB2.0" (id 1) (at 29.845 100.33 0))
-    (property "Footprint" "" (id 2) (at 33.655 120.65 0)
+    (property "Footprint" "HSD:USB-C-USB4105-GF-A-120" (id 2) (at 33.655 120.65 0)
       (effects (font (size 1.27 1.27)) hide)
     )
@@
     (property "Reference" "D4" (id 0) (at 87.9475 99.06 0))
     (property "Value" "SBA130CS_R1_00001" (id 1) (at 87.9475 101.6 0))
-    (property "Footprint" "" (id 2) (at 87.63 105.41 0)
+    (property "Footprint" "Diode_SMD:D_SOD-323" (id 2) (at 87.63 105.41 0)
       (effects (font (size 1.27 1.27)) hide)
     )
@@
     (property "Datasheet" "~" (id 3) (at 248.92 48.26 0)
       (effects (font (size 1.27 1.27)) hide)
-    )
-    (property "Voltage" "16V" (id 4) (at 252.73 52.07 0)
-      (effects (font (size 1.27 1.27)) (justify left))
     )
     (pin "1")
@@
       (effects (font (size 1.27 1.27)) hide)
     )
-    (property "Voltage" "6V3" (id 4) (at 199.39 52.07 0)
-      (effects (font (size 1.27 1.27)) (justify left))
-    )
     (pin "1")
     (pin "2")
@@
     (property "Reference" "L1" (id 0) (at 186.69 38.1 90))
     (property "Value" "2.2u" (id 1) (at 186.69 40.64 90))
-    (property "Footprint" "ppse_2021:Inductor" (id 2) (at 186.69 44.45 0)
+    (property "Footprint" "" (id 2) (at 186.69 44.45 0)
       (effects (font (size 1.27 1.27)) hide)
     )
     (property "Datasheet" "https://www.mouser.it/datasheet/2/54/SRP2512-1391417.pdf" (id 3) (at 186.69 44.45 0)
-      (effects (font (size 1.27 1.27)) hide)
-    )
-    (pin "1")
-    (pin "2")
-  )
-  (symbol (lib_id "Device:FerriteBead") (at 57.15 105.41 90) (unit 1)
-    (in_bom yes) (on_board yes) (fields_autoplaced)
-    (property "Reference" "FB1" (id 0) (at 57.0992 97.79 90))
-    (property "Value" "FerriteBead" (id 1) (at 57.0992 100.33 90))
-    (property "Footprint" "Inductor_SMD:L_0603_1608Metric" (id 2) (at 57.15 107.188 90)
-      (effects (font (size 1.27 1.27)) hide)
-    )
-    (property "Datasheet" "https://www.mouser.it/ProductDetail/Laird-Performance-Materials/LI0603E470R-10?qs=sGAEpiMZZMt1hubY80%2Fs8HXRixHmQiFc7i4a5UHD5sU%3D" (id 3) (at 57.15 105.41 0)
       (effects (font (size 1.27 1.27)) hide)
     )
@@
     (property "Reference" "F2" (id 0) (at 44.45 58.42 90))
     (property "Value" "C1T-T6" (id 1) (at 44.45 60.96 90))
-    (property "Footprint" "" (id 2) (at 44.45 66.548 90)
+    (property "Footprint" "Fuse:Fuse_1206_3216Metric" (id 2) (at 44.45 66.548 90)
       (effects (font (size 1.27 1.27)) hide)
     )
@@
       (effects (font (size 1.27 1.27)) (justify left))
     )
-    (property "Footprint" "Diode_SMD:D_SMA" (id 2) (at 52.07 68.58 0)
+    (property "Footprint" "Diode_SMD:D_SOD-123" (id 2) (at 52.07 68.58 0)
       (effects (font (size 1.27 1.27)) hide)
     )
@@
   (symbol (lib_id "Device:R") (at 48.895 110.49 90) (unit 1)
     (in_bom yes) (on_board yes)
-    (property "Reference" "R2" (id 0) (at 47.625 108.585 90))
-    (property "Value" "5k1" (id 1) (at 50.8 108.585 90))
-    (property "Footprint" "" (id 2) (at 48.895 112.268 90)
+    (property "Reference" "R2" (id 0) (at 48.26 107.95 90))
+    (property "Value" "5k1" (id 1) (at 49.53 110.49 90))
+    (property "Footprint" "Resistor_SMD:R_0603_1608Metric" (id 2) (at 48.895 112.268 90)
       (effects (font (size 1.27 1.27)) hide)
     )
@@
       (effects (font (size 1.27 1.27)) (justify left))
     )
-    (property "Footprint" "" (id 2) (at 20.447 147.32 90)
+    (property "Footprint" "Resistor_SMD:R_0603_1608Metric" (id 2) (at 20.447 147.32 90)
       (effects (font (size 1.27 1.27)) hide)
     )
@@
     (in_bom yes) (on_board yes)
     (property "Reference" "R3" (id 0) (at 47.625 115.57 90))
-    (property "Value" "5k1" (id 1) (at 50.8 115.57 90))
-    (property "Footprint" "" (id 2) (at 48.895 114.808 90)
+    (property "Value" "5k1" (id 1) (at 49.53 113.03 90))
+    (property "Footprint" "Resistor_SMD:R_0603_1608Metric" (id 2) (at 48.895 114.808 90)
       (effects (font (size 1.27 1.27)) hide)
     )
@@
     (property "Datasheet" "~" (id 3) (at 102.87 48.26 0)
       (effects (font (size 1.27 1.27)) hide)
-    )
-    (property "Voltage" "16V" (id 4) (at 106.68 52.07 0)
-      (effects (font (size 1.27 1.27)) (justify left))
     )
     (pin "1")
@@
     (in_bom yes) (on_board yes) (fields_autoplaced)
     (property "Reference" "D3" (id 0) (at 82.55 38.1 0))
-    (property "Value" "SMA S1B" (id 1) (at 82.55 40.64 0))
-    (property "Footprint" "Diode_SMD:D_SMA" (id 2) (at 82.55 40.005 0)
-      (effects (font (size 1.27 1.27)) hide)
-    )
-    (property "Datasheet" "https://www.diodes.com/assets/Datasheets/ds16003.pdf" (id 3) (at 82.55 44.45 0)
+    (property "Value" "GS1504FL" (id 1) (at 82.55 40.64 0))
+    (property "Footprint" "Diode_SMD:D_SOD-123F" (id 2) (at 82.55 40.005 0)
+      (effects (font (size 1.27 1.27)) hide)
+    )
+    (property "Datasheet" "https://www.mouser.it/datasheet/2/1057/GS1504FL_SERIES-1870309.pdf" (id 3) (at 82.55 44.45 0)
       (effects (font (size 1.27 1.27)) hide)
     )
@@
       (effects (font (size 1.27 1.27)) hide)
     )
-    (property "Voltage" "6V3" (id 4) (at 181.61 52.0701 0)
-      (effects (font (size 1.27 1.27)) (justify left))
-    )
     (pin "1")
     (pin "2")
@@
       (effects (font (size 1.27 1.27)) hide)
     )
-    (property "Tolerance" "1%" (id 4) (at 158.75 73.66 0)
-      (effects (font (size 1.27 1.27)) (justify left))
-    )
     (pin "1")
     (pin "2")
@@
       (effects (font (size 1.27 1.27)) hide)
     )
-    (property "Voltage" "16V" (id 4) (at 116.84 52.07 0)
-      (effects (font (size 1.27 1.27)) (justify left))
-    )
     (pin "1")
     (pin "2")
@@
     (in_bom yes) (on_board yes)
     (property "Reference" "F1" (id 0) (at 44.45 38.735 90))
-    (property "Value" "2929L-LF075" (id 1) (at 44.45 41.0464 90))
-    (property "Footprint" "" (id 2) (at 39.37 45.72 0)
+    (property "Value" "2920L075" (id 1) (at 44.45 41.0464 90))
+    (property "Footprint" "Fuse:Fuse_2920_7451Metric" (id 2) (at 39.37 45.72 0)
       (effects (font (size 1.27 1.27)) (justify left) hide)
     )
@@
       (effects (font (size 1.27 1.27)) hide)
     )
-    (property "Voltage" "16V" (id 4) (at 127 52.07 0)
-      (effects (font (size 1.27 1.27)) (justify left))
-    )
     (pin "1")
     (pin "2")
@@
       (effects (font (size 1.27 1.27)) hide)
     )
-    (property "Voltage" "16V" (id 4) (at 228.6 52.07 0)
-      (effects (font (size 1.27 1.27)) (justify left))
-    )
     (pin "1")
     (pin "2")
@@
       (effects (font (size 1.27 1.27)) hide)
     )
-    (property "Voltage" "6V3" (id 4) (at 209.55 52.07 0)
-      (effects (font (size 1.27 1.27)) (justify left))
-    )
-    (pin "1")
+    (pin "1")
