File: kicad-project/power.kicad_sch (KiCad schematic)
At the start: 32 parts, among them J1 Screw_Terminal_01x02, J2 USB_C_Receptacle_USB2.0, U1 TPS563201, U2 AMS1117-3.3

Commit message: hw: finish schematic, PS i2c R_pull-up wrong
Parts:
- removed FB1: FerriteBead, Inductor_SMD:L_0603_1608Metric, symbol Device:FerriteBead
- added R14: 10k, Resistor_SMD:R_0603_1608Metric, symbol Device:R
- C1, C2, C3, C7, C8: Voltage 16V -> (none)
- C4, C5, C6: Voltage 6V3 -> (none)
- D1: footprint (none) -> Diode_SMD:D_SOD-123
- D2: footprint Diode_SMD:D_SMA -> Diode_SMD:D_SOD-123
- D3: value SMA S1B -> GS1504FL; footprint Diode_SMD:D_SMA -> Diode_SMD:D_SOD-123F
- D4: footprint (none) -> Diode_SMD:D_SOD-323
- F1: value 2929L-LF075 -> 2920L075; footprint (none) -> Fuse:Fuse_2920_7451Metric
- F2: footprint (none) -> Fuse:Fuse_1206_3216Metric
- J1: footprint (none) -> TerminalBlock_RND:TerminalBlock_RND_205-00001_1x02_P5.00mm_Horizontal
- J2: footprint (none) -> HSD:USB-C-USB4105-GF-A-120
- L1: value 2.2u -> 4.7u; footprint ppse_2021:Inductor -> Inductor_SMD:L_0603_1608Metric
- R1, R2, R3: footprint (none) -> Resistor_SMD:R_0603_1608Metric
- R5: value 56k -> 56.2k; Tolerance 1% -> (none)
- U1: value TPS563201 -> AP62201WU-7; footprint Package_TO_SOT_SMD:SOT-23-6 -> Package_TO_SOT_SMD:TSOT-23-6
Connections:
- net VBUS_FILTERED is gone; now on net VBUS: D4.2 (A)
- net GND: now also R14.2
- net SW_EN: now also R14.1
Other:
- note added: "0603 C fino a 100n 0805 C da 1u in sù"
- note removed: "TUTTI I FOORPRINT SONO DA VERIFICARE/AGGIUNGERE"
