File: kicad-project/power.kicad_sch (KiCad schematic)
At the start: 32 parts, among them J1 Screw_Terminal_01x02, J2 USB_C_Receptacle_USB2.0, U1 AP62201WU-7, U2 AMS1117-3.3

Commit message: hw: place layout component
Parts:
- added R19: 0, Resistor_SMD:R_0603_1608Metric, symbol Device:R
- L1: value 4.7u -> (none); footprint Inductor_SMD:L_0603_1608Metric -> (none)
- R4: value 10k -> (none); footprint Resistor_SMD:R_0603_1608Metric -> (none)
Connections:
- net +5V: now also R19.1; no longer C7.1, U2.3 (VI)
- net GND: no longer R6.2
- net SW_FB: no longer R6.1
- new net: C7.1, R19.2, U2.3 (VI)
Other:
- moved on the sheet: R6
Changed lines of the file:
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@@
   (junction (at 96.52 44.45) (diameter 0) (color 0 0 0 0)
   )
+  (junction (at 224.79 44.45) (diameter 0) (color 0 0 0 0)
+  )
   (junction (at 143.51 49.53) (diameter 0) (color 0 0 0 0)
   )
@@
   )
   (junction (at 270.51 44.45) (diameter 0) (color 0 0 0 0)
-  )
-  (junction (at 214.63 44.45) (diameter 0) (color 0 0 0 0)
-  )
-  (junction (at 224.79 44.45) (diameter 0) (color 0 0 0 0)
   )
   (junction (at 46.355 120.65) (diameter 0) (color 0 0 0 0)
@@
     (stroke (width 0) (type default) (color 0 0 0 0))
   )
-  (wire (pts (xy 205.74 44.45) (xy 214.63 44.45))
-    (stroke (width 0) (type default) (color 0 0 0 0))
-  )
   (wire (pts (xy 48.26 44.45) (xy 57.15 44.45))
     (stroke (width 0) (type default) (color 0 0 0 0))
@@
     (stroke (width 0) (type default) (color 0 0 0 0))
   )
-  (wire (pts (xy 214.63 44.45) (xy 224.79 44.45))
-    (stroke (width 0) (type default) (color 0 0 0 0))
-  )
   (wire (pts (xy 96.52 105.41) (xy 96.52 44.45))
     (stroke (width 0) (type default) (color 0 0 0 0))
@@
     (stroke (width 0) (type default) (color 0 0 0 0))
   )
+  (wire (pts (xy 205.74 44.45) (xy 212.09 44.45))
+    (stroke (width 0) (type default) (color 0 0 0 0))
+  )
   (wire (pts (xy 224.79 44.45) (xy 229.87 44.45))
     (stroke (width 0) (type default) (color 0 0 0 0))
@@
   )
   (wire (pts (xy 130.81 49.53) (xy 132.08 49.53))
+    (stroke (width 0) (type default) (color 0 0 0 0))
+  )
+  (wire (pts (xy 219.71 44.45) (xy 224.79 44.45))
     (stroke (width 0) (type default) (color 0 0 0 0))
   )
@@
     (pin "1")
   )
+  (symbol (lib_id "Device:R") (at 215.9 44.45 90) (unit 1)
+    (in_bom yes) (on_board yes) (fields_autoplaced)
+    (property "Reference" "R19" (id 0) (at 215.9 38.1 90))
+    (property "Value" "0" (id 1) (at 215.9 40.64 90))
+    (property "Footprint" "Resistor_SMD:R_0603_1608Metric" (id 2) (at 215.9 46.228 90)
+      (effects (font (size 1.27 1.27)) hide)
+    )
+    (property "Datasheet" "~" (id 3) (at 215.9 44.45 0)
+      (effects (font (size 1.27 1.27)) hide)
+    )
+    (pin "1")
+    (pin "2")
+  )
   (symbol (lib_id "Connector:Screw_Terminal_01x02") (at 21.59 46.99 180) (unit 1)
     (in_bom yes) (on_board yes) (fields_autoplaced)
@@
     (pin "1")
   )
-  (symbol (lib_id "power:+5V") (at 214.63 44.45 0) (unit 1)
+  (symbol (lib_id "power:+5V") (at 205.74 44.45 0) (unit 1)
     (in_bom yes) (on_board yes) (fields_autoplaced)
-    (property "Reference" "#PWR016" (id 0) (at 214.63 48.26 0)
-      (effects (font (size 1.27 1.27)) hide)
-    )
-    (property "Value" "+5V" (id 1) (at 214.63 39.37 0))
-    (property "Footprint" "" (id 2) (at 214.63 44.45 0)
-      (effects (font (size 1.27 1.27)) hide)
-    )
-    (property "Datasheet" "" (id 3) (at 214.63 44.45 0)
-      (effects (font (size 1.27 1.27)) hide)
-    )
-    (pin "1")
-  )
-  (symbol (lib_id "Device:R") (at 157.48 81.28 0) (unit 1)
-    (in_bom yes) (on_board yes)
-    (property "Reference" "R6" (id 0) (at 158.75 78.74 0)
+    (property "Reference" "#PWR016" (id 0) (at 205.74 48.26 0)
+      (effects (font (size 1.27 1.27)) hide)
+    )
+    (property "Value" "+5V" (id 1) (at 205.74 39.37 0))
+    (property "Footprint" "" (id 2) (at 205.74 44.45 0)
+      (effects (font (size 1.27 1.27)) hide)
+    )
+    (property "Datasheet" "" (id 3) (at 205.74 44.45 0)
+      (effects (font (size 1.27 1.27)) hide)
+    )
+    (pin "1")
+  )
+  (symbol (lib_id "Device:R") (at 157.48 81.28 90) (unit 1)
+    (in_bom yes) (on_board yes)
+    (property "Reference" "R6" (id 0) (at 154.94 80.01 0)
       (effects (font (size 1.27 1.27)) (justify left))
     )
-    (property "Value" "10k" (id 1) (at 158.75 81.28 0)
+    (property "Value" "10k" (id 1) (at 157.48 80.01 0)
       (effects (font (size 1.27 1.27)) (justify left))
     )
-    (property "Footprint" "Resistor_SMD:R_0603_1608Metric" (id 2) (at 155.702 81.28 90)
+    (property "Footprint" "Resistor_SMD:R_0603_1608Metric" (id 2) (at 157.48 83.058 90)
       (effects (font (size 1.27 1.27)) hide)
     )
@@
     (in_bom yes) (on_board yes) (fields_autoplaced)
     (property "Reference" "L1" (id 0) (at 186.69 38.1 90))
-    (property "Value" "4.7u" (id 1) (at 186.69 40.64 90))
-    (property "Footprint" "Inductor_SMD:L_0603_1608Metric" (id 2) (at 186.69 44.45 0)
+    (property "Value" "" (id 1) (at 186.69 40.64 90))
+    (property "Footprint" "" (id 2) (at 186.69 44.45 0)
       (effects (font (size 1.27 1.27)) hide)
     )
@@
     (in_bom yes) (on_board yes)
     (property "Reference" "R4" (id 0) (at 135.89 52.07 90))
-    (property "Value" "10k" (id 1) (at 135.89 54.61 90))
-    (property "Footprint" "Resistor_SMD:R_0603_1608Metric" (id 2) (at 135.89 51.308 90)
-      (effects (font (size 1.27 1.27)) hide)
-    )
+    (property "Value" "" (id 1) (at 135.89 54.61 90))
+    (property "Footprint" "" (id 2) (at 135.89 51.308 90)
+      (effects (font (size 1.27 1.27)) hide)
+    )

Commit message: fix unipolar e qualche rotta
Parts:
- L1: value (none) -> 4.7u; footprint (none) -> HSD:Inductance
- R4: value (none) -> 10k; footprint (none) -> Resistor_SMD:R_0603_1608Metric
Changed lines of the file:
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@@
     (in_bom yes) (on_board yes) (fields_autoplaced)
     (property "Reference" "L1" (id 0) (at 186.69 38.1 90))
-    (property "Value" "" (id 1) (at 186.69 40.64 90))
-    (property "Footprint" "" (id 2) (at 186.69 44.45 0)
+    (property "Value" "4.7u" (id 1) (at 186.69 40.64 90))
+    (property "Footprint" "HSD:Inductance" (id 2) (at 186.69 44.45 0)
       (effects (font (size 1.27 1.27)) hide)
     )
@@
     (in_bom yes) (on_board yes)
     (property "Reference" "R4" (id 0) (at 135.89 52.07 90))
-    (property "Value" "" (id 1) (at 135.89 54.61 90))
-    (property "Footprint" "" (id 2) (at 135.89 51.308 90)
-      (effects (font (size 1.27 1.27)) hide)
-    )
+    (property "Value" "10k" (id 1) (at 135.89 54.61 90))
+    (property "Footprint" "Resistor_SMD:R_0603_1608Metric" (id 2) (at 135.89 51.308 90)
+      (effects (font (size 1.27 1.27)) hide)
+    )

Commit message: hw: HSD v1.0 w/out peripherals
Connections:
- net GND: now also R6.1
- net SW_FB: now also R6.2
Other:
- moved on the sheet: R6
Changed lines of the file:
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@@
     (pin "1")
   )
-  (symbol (lib_id "power:+5V") (at 205.74 44.45 0) (unit 1)
+  (symbol (lib_id "power:+5V") (at 205.74 44.45 0) (mirror y) (unit 1)
     (in_bom yes) (on_board yes) (fields_autoplaced)
     (property "Reference" "#PWR016" (id 0) (at 205.74 48.26 0)
@@
     (pin "1")
   )
-  (symbol (lib_id "Device:R") (at 157.48 81.28 90) (unit 1)
+  (symbol (lib_id "Device:R") (at 157.48 81.28 180) (unit 1)
     (in_bom yes) (on_board yes)
-    (property "Reference" "R6" (id 0) (at 154.94 80.01 0)
+    (property "Reference" "R6" (id 0) (at 156.21 83.82 0)
       (effects (font (size 1.27 1.27)) (justify left))
     )
-    (property "Value" "10k" (id 1) (at 157.48 80.01 0)
+    (property "Value" "10k" (id 1) (at 156.21 81.28 0)
       (effects (font (size 1.27 1.27)) (justify left))
     )
-    (property "Footprint" "Resistor_SMD:R_0603_1608Metric" (id 2) (at 157.48 83.058 90)
+    (property "Footprint" "Resistor_SMD:R_0603_1608Metric" (id 2) (at 159.258 81.28 90)
       (effects (font (size 1.27 1.27)) hide)
     )
