File: kicad-project/rp2040.kicad_sch (KiCad schematic)
At the start: 29 parts, among them SW1 PRG_SW, SW2 RST_SW, SW3 EN_SW, U3 RP2040, U4 W25Q16JVSS, Y1 16MHz

Commit message: hw: finish schematic
Parts:
- added C34: 100n, Capacitor_SMD:C_0603_1608Metric, symbol Device:C
- added R42, R43: 10k, Resistor_SMD:R_0603_1608Metric, symbol Device:R
- C21, C22: value 22p -> 27p
- C23, C9: Voltage 6V3 -> (none)
- R12: value DNP 10k -> 10k DNP
- R13: value 1M -> 1k
- SW1, SW2: footprint Button_Switch_THT:SW_PUSH_6mm -> Button_Switch_SMD:SW_Push_1P1T_NO_CK_KMR2
- SW3: value EN_SW -> EN_BTN; footprint Button_Switch_THT:SW_PUSH_6mm -> Button_Switch_SMD:SW_Push_1P1T_NO_CK_KMR2
- Y1: value 16MHz -> ABLS-12.000MHz
Connections:
- net BUZZER: now also U3.4 (GPIO2); no longer U3.2 (GPIO0)
- net DIR_A: now also U3.12 (GPIO9); no longer U3.9 (GPIO7)
- net DIR_B: now also U3.14 (GPIO11); no longer U3.12 (GPIO9)
- net DIR_C: now also U3.16 (GPIO13); no longer U3.14 (GPIO11)
- net DIR_D: now also U3.18 (GPIO15); no longer U3.16 (GPIO13)
- net EN_MOTORS: now also U3.9 (GPIO7); no longer U3.7 (GPIO5)
- net ESP_RX: now also U3.3 (GPIO1); no longer U3.35 (GPIO23)
- net ESP_TX: now also U3.2 (GPIO0); no longer U3.34 (GPIO22)
- net GND: now also C34.2, R42.2, R43.2
- net I2C_SCL: now also R42.1
- net I2C_SDA: now also R43.1
- net LED_B: now also U3.7 (GPIO5); no longer U3.5 (GPIO3)
- net LED_G: now also U3.5 (GPIO3); no longer U3.3 (GPIO1)
- net LED_R: now also U3.6 (GPIO4); no longer U3.4 (GPIO2)
- net LS1: now also U3.31 (GPIO20); no longer U3.29 (GPIO18)
- net LS2: now also U3.32 (GPIO21); no longer U3.30 (GPIO19)
- net LS3: now also U3.34 (GPIO22); no longer U3.31 (GPIO20)
- net LS4: now also U3.35 (GPIO23); no longer U3.32 (GPIO21)
- net ME_W11: now also U3.27 (GPIO16); no longer U3.17 (GPIO14)
- net ME_W12: now also U3.28 (GPIO17); no longer U3.18 (GPIO15)
- net ME_W21: now also U3.29 (GPIO18); no longer U3.27 (GPIO16)
- net ME_W22: now also U3.30 (GPIO19); no longer U3.28 (GPIO17)
- net STEP_A: now also U3.11 (GPIO8); no longer U3.8 (GPIO6)
- net STEP_B: now also U3.13 (GPIO10); no longer U3.11 (GPIO8)
- net STEP_C: now also U3.15 (GPIO12); no longer U3.13 (GPIO10)
- net STEP_D: now also U3.17 (GPIO14); no longer U3.15 (GPIO12)
- net ~{RESET}: now also C34.1
- net ~{EN_SW} renamed ~{EN_BTN}
- net ~{EN_BTN}: now also U3.8 (GPIO6); no longer U3.6 (GPIO4)
Other:
- note added: "Motors Enable Toggle"
- note added: "Place R close to rp2040 pins"
- note removed: "Motor Enable Switch"
- note removed: "Place R_{termination} close to rp2040 pins"
- moved on the sheet: R10, SW2
