File: kicad-project/rp2040.kicad_sch (KiCad schematic)
At the start: 33 parts, among them J3 Conn_02x04_Odd_Even, SW1 PRG_SW, SW2 RST_SW, SW3 ESP_RST_SW, U3 RP2040, U4 W25Q16JVSS, Y1 ABLS-12.000MHz

Commit message: hw: place layout component
Changed lines of the file:
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@@
-    (pin "1")
-  )
-  (symbol (lib_id "power:GND") (at 200.66 115.57 0) (unit 1)
-    (in_bom yes) (on_board yes)
-    (property "Reference" "#PWR0101" (id 0) (at 200.66 121.92 0)
-      (effects (font (size 1.27 1.27)) hide)
-    )
-    (property "Value" "GND" (id 1) (at 200.787 119.9642 0))
-    (property "Footprint" "" (id 2) (at 200.66 115.57 0)
-      (effects (font (size 1.27 1.27)) hide)
-    )
-    (property "Datasheet" "" (id 3) (at 200.66 115.57 0)
-      (effects (font (size 1.27 1.27)) hide)
-    )
     (pin "1")
   )

Commit message: hw: HSD v1.0 w/out peripherals
Parts:
- added D6: GREEN_LED, LED_SMD:LED_0603_1608Metric, symbol Device:LED
- added R20: 330, Resistor_SMD:R_0603_1608Metric, symbol Device:R
Connections:
- net DIR_A: now also U3.7 (GPIO5); no longer U3.12 (GPIO9)
- net DIR_B: now also U3.8 (GPIO6); no longer U3.14 (GPIO11)
- net DIR_C: now also U3.5 (GPIO3); no longer U3.16 (GPIO13)
- net DIR_D: now also U3.2 (GPIO0); no longer U3.18 (GPIO15)
- net EN_MOTORS: now also U3.4 (GPIO2); no longer U3.9 (GPIO7)
- net ESP_RX: no longer R15.1, U3.2 (GPIO0)
- net GND: now also R20.2
- net LS1: now also U3.36 (GPIO24); no longer U3.31 (GPIO20)
- net LS2: now also U3.37 (GPIO25); no longer U3.32 (GPIO21)
- net LS3: now also U3.38 (GPIO26/ADC0); no longer U3.34 (GPIO22)
- net LS4: now also U3.39 (GPIO27/ADC1); no longer U3.35 (GPIO23)
- net ME_W11: now also U3.30 (GPIO19); no longer U3.27 (GPIO16)
- net ME_W12: now also U3.31 (GPIO20); no longer U3.28 (GPIO17)
- net ME_W21: now also U3.32 (GPIO21); no longer U3.29 (GPIO18)
- net ME_W22: now also U3.34 (GPIO22); no longer U3.30 (GPIO19)
- net STEP_A: now also U3.9 (GPIO7); no longer U3.11 (GPIO8)
- net STEP_B: now also U3.11 (GPIO8); no longer U3.13 (GPIO10)
- net STEP_C: now also U3.6 (GPIO4); no longer U3.15 (GPIO12)
- net STEP_D: now also U3.3 (GPIO1); no longer U3.17 (GPIO14)
- net at U3.41 (GPIO29/ADC3): now also D6.2 (A)
- net ESP_TX renamed MCU_UART0_RX
- net MCU_UART0_RX: now also U3.17 (GPIO14); no longer U3.3 (GPIO1)
- new net: D6.1 (K), R20.1
- new net MCU_UART0_TX: R15.1, U3.16 (GPIO13)
