File: kicad-project/unipolar.kicad_sch (KiCad schematic)
At the start: 17 parts

Commit message: hw: update to complete schematic
Parts:
- D7: renamed from D?; value CGRA4007 -> RB160QS-40T18R; footprint Diode_SMD:D_SMA -> (none)
- gave numbers to parts that had none: 16
Connections:
- net +12V: no longer D7.1 (K), J21.1 (Pin_1)
- net M1_W11 renamed ME_W11
- net M1_W12 renamed ME_W12
- net M1_W21 renamed ME_W21
- net M1_W22 renamed ME_W22
- new net +5V: D7.1 (K), J21.1 (Pin_1)
Other:
- note added: "Unipolar ME"
- note removed: "Stepper Driver 1"
- note removed: "Stepper Motors"
- note removed: "Unipolar stepper motor 28BYJ (ADAFRUIT 918) 12V version"
- moved on the sheet: J21

Commit message: hw: finish schematic
Parts:
- D10, D8, D9: value CGRA4007 -> 1N4148WS; footprint Diode_SMD:D_SMA -> Diode_SMD:D_SOD-323
- D7: value RB160QS-40T18R -> 1N4148WS; footprint (none) -> Diode_SMD:D_SOD-323
- J21: footprint Connector_JST:JST_XH_S5B-XH-A_1x05_P2.50mm_Horizontal -> Connector_JST:JST_XH_B5B-XH-AM_1x05_P2.50mm_Vertical
- Q5, Q6, Q7, Q8: value SI2300DS -> 2N7002NXAKR; symbol Device:Q_NMOS_DGS -> Device:Q_NMOS_GSD
Connections:
- net GND: now also Q5.2 (S), Q6.2 (S), Q7.2 (S), Q8.2 (S); no longer Q5.3 (S), Q6.3 (S), Q7.3 (S), Q8.3 (S)
- net M1_OUT1: now also Q5.3 (D); no longer Q5.1 (D)
- net M1_OUT2: now also Q6.3 (D); no longer Q6.1 (D)
- net M1_OUT3: now also Q7.3 (D); no longer Q7.1 (D)
- net M1_OUT4: now also Q8.3 (D); no longer Q8.1 (D)
- net at R37.2, R41.1: now also Q8.1 (G); no longer Q8.2 (G)
- net at R36.2, R40.1: now also Q7.1 (G); no longer Q7.2 (G)
- net at R34.2, R38.1: now also Q5.1 (G); no longer Q5.2 (G)
- net at R35.2, R39.1: now also Q6.1 (G); no longer Q6.2 (G)

Commit message: fix unipolar e qualche rotta
Parts:
- Q5: value 2N7002NXAKR -> (none); footprint Package_TO_SOT_SMD:SOT-23 -> (none)
Connections:
- net +12V is gone; now on net +5V: D10.1 (K), D8.1 (K), D9.1 (K)
Changed lines of the file:
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@@
-    (pin "1")
-  )
-  (symbol (lib_id "power:+12V") (at 58.42 77.47 0) (unit 1)
-    (in_bom yes) (on_board yes) (fields_autoplaced)
-    (property "Reference" "#PWR0121" (id 0) (at 58.42 81.28 0)
-      (effects (font (size 1.27 1.27)) hide)
-    )
-    (property "Value" "+12V" (id 1) (at 58.42 72.39 0))
-    (property "Footprint" "" (id 2) (at 58.42 77.47 0)
-      (effects (font (size 1.27 1.27)) hide)
-    )
-    (property "Datasheet" "" (id 3) (at 58.42 77.47 0)
-      (effects (font (size 1.27 1.27)) hide)
-    )
     (pin "1")
   )
@@
       (effects (font (size 1.27 1.27)) (justify left))
     )
-    (property "Value" "2N7002NXAKR" (id 1) (at 62.23 57.1499 0)
-      (effects (font (size 1.27 1.27)) (justify left))
-    )
-    (property "Footprint" "Package_TO_SOT_SMD:SOT-23" (id 2) (at 60.96 53.34 0)
+    (property "Value" "" (id 1) (at 62.23 57.1499 0)
+      (effects (font (size 1.27 1.27)) (justify left))
+    )
+    (property "Footprint" "" (id 2) (at 60.96 53.34 0)
       (effects (font (size 1.27 1.27)) hide)
     )
@@
     (pin "3")
   )
+  (symbol (lib_id "power:+5V") (at 58.42 77.47 0) (unit 1)
+    (in_bom yes) (on_board yes) (fields_autoplaced)
+    (property "Reference" "#PWR?" (id 0) (at 58.42 81.28 0)
+      (effects (font (size 1.27 1.27)) hide)
+    )
+    (property "Value" "+5V" (id 1) (at 58.42 72.39 0))
+    (property "Footprint" "" (id 2) (at 58.42 77.47 0)
+      (effects (font (size 1.27 1.27)) hide)
+    )
+    (property "Datasheet" "" (id 3) (at 58.42 77.47 0)
+      (effects (font (size 1.27 1.27)) hide)
+    )
+    (pin "1")
+  )
   (symbol (lib_id "power:GND") (at 58.42 133.35 0) (unit 1)
     (in_bom yes) (on_board yes) (fields_autoplaced)
@@
     (pin "2")
   )
-  (symbol (lib_id "power:+12V") (at 58.42 113.03 0) (unit 1)
-    (in_bom yes) (on_board yes) (fields_autoplaced)
-    (property "Reference" "#PWR0123" (id 0) (at 58.42 116.84 0)
-      (effects (font (size 1.27 1.27)) hide)
-    )
-    (property "Value" "+12V" (id 1) (at 58.42 107.95 0))
+  (symbol (lib_id "Device:R") (at 49.53 129.54 0) (unit 1)
+    (in_bom yes) (on_board yes) (fields_autoplaced)
+    (property "Reference" "R40" (id 0) (at 52.07 128.2699 0)
+      (effects (font (size 1.27 1.27)) (justify left))
+    )
+    (property "Value" "10k" (id 1) (at 52.07 130.8099 0)
+      (effects (font (size 1.27 1.27)) (justify left))
+    )
+    (property "Footprint" "Resistor_SMD:R_0603_1608Metric" (id 2) (at 47.752 129.54 90)
+      (effects (font (size 1.27 1.27)) hide)
+    )
+    (property "Datasheet" "~" (id 3) (at 49.53 129.54 0)
+      (effects (font (size 1.27 1.27)) hide)
+    )
+    (pin "1")
+    (pin "2")
+  )
+  (symbol (lib_id "Device:R") (at 49.53 59.69 0) (unit 1)
+    (in_bom yes) (on_board yes) (fields_autoplaced)
+    (property "Reference" "R38" (id 0) (at 52.07 58.4199 0)
+      (effects (font (size 1.27 1.27)) (justify left))
+    )
+    (property "Value" "10k" (id 1) (at 52.07 60.9599 0)
+      (effects (font (size 1.27 1.27)) (justify left))
+    )
+    (property "Footprint" "Resistor_SMD:R_0603_1608Metric" (id 2) (at 47.752 59.69 90)
+      (effects (font (size 1.27 1.27)) hide)
+    )
+    (property "Datasheet" "~" (id 3) (at 49.53 59.69 0)
+      (effects (font (size 1.27 1.27)) hide)
+    )
+    (pin "1")
+    (pin "2")
+  )
+  (symbol (lib_id "power:+5V") (at 58.42 149.86 0) (unit 1)
+    (in_bom yes) (on_board yes) (fields_autoplaced)
+    (property "Reference" "#PWR?" (id 0) (at 58.42 153.67 0)
+      (effects (font (size 1.27 1.27)) hide)
+    )
+    (property "Value" "+5V" (id 1) (at 58.42 144.78 0))
+    (property "Footprint" "" (id 2) (at 58.42 149.86 0)
+      (effects (font (size 1.27 1.27)) hide)
+    )
+    (property "Datasheet" "" (id 3) (at 58.42 149.86 0)
+      (effects (font (size 1.27 1.27)) hide)
+    )
+    (pin "1")
+  )
+  (symbol (lib_id "Device:D") (at 58.42 153.67 270) (unit 1)
+    (in_bom yes) (on_board yes) (fields_autoplaced)
+    (property "Reference" "D10" (id 0) (at 60.96 152.3999 90)
+      (effects (font (size 1.27 1.27)) (justify left))
+    )
+    (property "Value" "1N4148WS" (id 1) (at 60.96 154.9399 90)
+      (effects (font (size 1.27 1.27)) (justify left))
+    )
+    (property "Footprint" "Diode_SMD:D_SOD-323" (id 2) (at 58.42 153.67 0)
+      (effects (font (size 1.27 1.27)) hide)
+    )
+    (property "Datasheet" "https://www.mouser.it/datasheet/2/1057/1N4148WS-1869723.pdf" (id 3) (at 58.42 153.67 0)
+      (effects (font (size 1.27 1.27)) hide)
+    )
+    (pin "1")
+    (pin "2")
+  )
+  (symbol (lib_id "Device:Q_NMOS_GSD") (at 55.88 90.17 0) (unit 1)
+    (in_bom yes) (on_board yes) (fields_autoplaced)
+    (property "Reference" "Q6" (id 0) (at 62.23 88.8999 0)
+      (effects (font (size 1.27 1.27)) (justify left))
+    )
+    (property "Value" "2N7002NXAKR" (id 1) (at 62.23 91.4399 0)
+      (effects (font (size 1.27 1.27)) (justify left))
+    )
+    (property "Footprint" "Package_TO_SOT_SMD:SOT-23" (id 2) (at 60.96 87.63 0)
+      (effects (font (size 1.27 1.27)) hide)
+    )
+    (property "Datasheet" "~" (id 3) (at 55.88 90.17 0)
+      (effects (font (size 1.27 1.27)) hide)
+    )
+    (pin "1")
+    (pin "2")
+    (pin "3")
+  )
+  (symbol (lib_id "power:+5V") (at 58.42 113.03 0) (unit 1)
+    (in_bom yes) (on_board yes) (fields_autoplaced)
+    (property "Reference" "#PWR?" (id 0) (at 58.42 116.84 0)
+      (effects (font (size 1.27 1.27)) hide)
+    )
+    (property "Value" "+5V" (id 1) (at 58.42 107.95 0))
     (property "Footprint" "" (id 2) (at 58.42 113.03 0)
       (effects (font (size 1.27 1.27)) hide)
@@
     )
     (pin "1")
-  )
-  (symbol (lib_id "Device:R") (at 49.53 129.54 0) (unit 1)
-    (in_bom yes) (on_board yes) (fields_autoplaced)
-    (property "Reference" "R40" (id 0) (at 52.07 128.2699 0)
-      (effects (font (size 1.27 1.27)) (justify left))
-    )
-    (property "Value" "10k" (id 1) (at 52.07 130.8099 0)
-      (effects (font (size 1.27 1.27)) (justify left))
-    )
-    (property "Footprint" "Resistor_SMD:R_0603_1608Metric" (id 2) (at 47.752 129.54 90)
-      (effects (font (size 1.27 1.27)) hide)
-    )
-    (property "Datasheet" "~" (id 3) (at 49.53 129.54 0)
-      (effects (font (size 1.27 1.27)) hide)
-    )
-    (pin "1")
-    (pin "2")
-  )
-  (symbol (lib_id "Device:R") (at 49.53 59.69 0) (unit 1)
-    (in_bom yes) (on_board yes) (fields_autoplaced)
-    (property "Reference" "R38" (id 0) (at 52.07 58.4199 0)
-      (effects (font (size 1.27 1.27)) (justify left))
-    )
-    (property "Value" "10k" (id 1) (at 52.07 60.9599 0)
-      (effects (font (size 1.27 1.27)) (justify left))
-    )
-    (property "Footprint" "Resistor_SMD:R_0603_1608Metric" (id 2) (at 47.752 59.69 90)
-      (effects (font (size 1.27 1.27)) hide)
-    )
-    (property "Datasheet" "~" (id 3) (at 49.53 59.69 0)
-      (effects (font (size 1.27 1.27)) hide)
-    )
-    (pin "1")
-    (pin "2")
-  )
-  (symbol (lib_id "Device:D") (at 58.42 153.67 270) (unit 1)
-    (in_bom yes) (on_board yes) (fields_autoplaced)
-    (property "Reference" "D10" (id 0) (at 60.96 152.3999 90)
-      (effects (font (size 1.27 1.27)) (justify left))
-    )
-    (property "Value" "1N4148WS" (id 1) (at 60.96 154.9399 90)
-      (effects (font (size 1.27 1.27)) (justify left))
-    )
-    (property "Footprint" "Diode_SMD:D_SOD-323" (id 2) (at 58.42 153.67 0)
-      (effects (font (size 1.27 1.27)) hide)
-    )
-    (property "Datasheet" "https://www.mouser.it/datasheet/2/1057/1N4148WS-1869723.pdf" (id 3) (at 58.42 153.67 0)
-      (effects (font (size 1.27 1.27)) hide)
-    )
-    (pin "1")
-    (pin "2")
-  )
-  (symbol (lib_id "Device:Q_NMOS_GSD") (at 55.88 90.17 0) (unit 1)
-    (in_bom yes) (on_board yes) (fields_autoplaced)
-    (property "Reference" "Q6" (id 0) (at 62.23 88.8999 0)
-      (effects (font (size 1.27 1.27)) (justify left))
-    )
-    (property "Value" "2N7002NXAKR" (id 1) (at 62.23 91.4399 0)
-      (effects (font (size 1.27 1.27)) (justify left))
-    )
-    (property "Footprint" "Package_TO_SOT_SMD:SOT-23" (id 2) (at 60.96 87.63 0)
-      (effects (font (size 1.27 1.27)) hide)
-    )
-    (property "Datasheet" "~" (id 3) (at 55.88 90.17 0)
-      (effects (font (size 1.27 1.27)) hide)
-    )
-    (pin "1")
-    (pin "2")
-    (pin "3")
   )
   (symbol (lib_id "power:GND") (at 58.42 97.79 0) (unit 1)
@@
     (pin "2")
   )
-  (symbol (lib_id "power:+12V") (at 58.42 149.86 0) (unit 1)
-    (in_bom yes) (on_board yes) (fields_autoplaced)
-    (property "Reference" "#PWR0125" (id 0) (at 58.42 153.67 0)
-      (effects (font (size 1.27 1.27)) hide)
-    )
-    (property "Value" "+12V" (id 1) (at 58.42 144.78 0))
-    (property "Footprint" "" (id 2) (at 58.42 149.86 0)
-      (effects (font (size 1.27 1.27)) hide)
-    )
-    (property "Datasheet" "" (id 3) (at 58.42 149.86 0)
-      (effects (font (size 1.27 1.27)) hide)
-    )
-    (pin "1")
-  )
   (symbol (lib_id "Device:R") (at 49.53 93.98 0) (unit 1)

Commit message: hw: HSD v1.0 w/out peripherals
Parts:
- Q5: value (none) -> 2N7002NXAKR; footprint (none) -> Package_TO_SOT_SMD:SOT-23
Changed lines of the file:
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@@
       (effects (font (size 1.27 1.27)) (justify left))
     )
-    (property "Value" "" (id 1) (at 62.23 57.1499 0)
+    (property "Value" "2N7002NXAKR" (id 1) (at 62.23 57.1499 0)
       (effects (font (size 1.27 1.27)) (justify left))
     )
-    (property "Footprint" "" (id 2) (at 60.96 53.34 0)
+    (property "Footprint" "Package_TO_SOT_SMD:SOT-23" (id 2) (at 60.96 53.34 0)
       (effects (font (size 1.27 1.27)) hide)
     )
@@
   (symbol (lib_id "power:+5V") (at 58.42 77.47 0) (unit 1)
     (in_bom yes) (on_board yes) (fields_autoplaced)
-    (property "Reference" "#PWR?" (id 0) (at 58.42 81.28 0)
+    (property "Reference" "#PWR0103" (id 0) (at 58.42 81.28 0)
       (effects (font (size 1.27 1.27)) hide)
     )
@@
   (symbol (lib_id "power:+5V") (at 58.42 149.86 0) (unit 1)
     (in_bom yes) (on_board yes) (fields_autoplaced)
-    (property "Reference" "#PWR?" (id 0) (at 58.42 153.67 0)
+    (property "Reference" "#PWR0102" (id 0) (at 58.42 153.67 0)
       (effects (font (size 1.27 1.27)) hide)
     )
@@
   (symbol (lib_id "power:+5V") (at 58.42 113.03 0) (unit 1)
     (in_bom yes) (on_board yes) (fields_autoplaced)
-    (property "Reference" "#PWR?" (id 0) (at 58.42 116.84 0)
+    (property "Reference" "#PWR0101" (id 0) (at 58.42 116.84 0)
       (effects (font (size 1.27 1.27)) hide)
     )
